Commit message: gripper accomodation in urdf and srdf

File: ros_ur_driver/Universal_Robots_ROS2_Description/urdf/ur_macro.xacro (robot description, xacro)
@@ -438,6 +438,6 @@
       <child link="${tf_prefix}tool0"/>
     </joint>
-    <!-- commented for project -->
-    <!-- <link name="virtual_jaw_edge"/>
+    <!-- custom accomodation for gripper -->
+    <link name="virtual_jaw_edge"/>
     <joint name="Virtual_jaw_joint" type="fixed">
         <parent link="${tf_prefix}tool0"/>
@@ -450,5 +450,5 @@
         <child link="virtual_camera"/>
         <origin xyz="-0.06 0.0158 0.079" rpy="0 0 0"/>
-    </joint> -->
+    </joint>
   </xacro:macro>
 </robot>

File: ros_ur_driver/Universal_Robots_ROS2_Driver/ur_moveit_config/srdf/ur_macro.srdf.xacro (robot description, xacro)
@@ -12,5 +12,5 @@
     <!--SUBGROUPS - Groups can also be formed by referencing to already defined group names-->
     <group name="${prefix}${name}_manipulator">
-      <chain base_link="${prefix}base_link" tip_link="${prefix}tool0" />
+      <chain base_link="${prefix}base_link" tip_link="${prefix}virtual_jaw_edge" />
     </group>
     <!--GROUP STATES - Purpose - Define a named state for a particular group, in terms of joint values. This is useful to define states like 'folded arms'-->
